File: Hardware/Papa_Soundie_doublesided.brd (EAGLE design)
At the start: 38.1 x 63.5 mm, 79 parts, among them J1 Audio Jack, J2 MICRO-SD_CARD_SOCKET, U1 ATMEGA328P_TQFP, U2 VS1000D, U3 3.3V, U4 4MB Flash, Y1 12MHz, Y2 8MHz

Commit message: trying something new
Parts:
- J6: device SparkFun-Connectors:1X07 -> SparkFun-Connectors:1X05
- J8: device SparkFun-Connectors:1X04 -> SparkFun-Connectors:1X02
- moved C13 50.9 mm to (28.6, 69.2)
- moved C7 50.0 mm to (-25.4, 68.9), turned to 90 degrees
- moved J7 48.5 mm to (1.27, 44.5)
- moved S1 41.1 mm to (-6.67, 70.5)
- moved C16 41.0 mm to (-6.03, 65.2)
- moved D1 41.0 mm to (-6.03, 61.6)
- moved R17 41.0 mm to (-6.03, 63.3)
- moved J8 39.8 mm to (1.27, 57.1), turned to 270 degrees
- moved J5 38.7 mm to (36.8, 31.8), turned to 90 degrees
- moved J10 37.8 mm to (36.8, 26.7)
- moved J11 37.8 mm to (36.8, 21.6)
- moved J3 37.8 mm to (36.8, 16.5)
- moved R15 36.6 mm to (-11.7, 63.0), turned to 180 degrees
- moved C3 35.6 mm to (-23.7, 78.1), turned to 90 degrees
- moved C6 33.8 mm to (-11.7, 61.1), turned to 0 degrees
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Connections:
- removed net A2: J8.3, U1.25
- removed net A3: J8.4, U1.26
- removed net D7: J6.7, U1.11
- removed net D8: J6.6, U1.12
- net USBN: now also J10.2; no longer J10.1
- net USBP: now also J10.1; no longer J10.2
- net VS_RX: now also J11.2; no longer J11.1
- net VS_TX: now also J11.1; no longer J11.2
Routing:
- net VCC: track 69.4 -> 0.00 mm, vias 4 -> 0
- net SCL: track 66.5 -> 0.00 mm, vias 1 -> 0
- net SDA: track 60.1 -> 0.00 mm, vias 1 -> 0
- net L_AC: track 57.1 -> 0.00 mm, vias 1 -> 0
- net R_AC: track 44.7 -> 0.00 mm, vias 1 -> 0
- net DVDD: track 43.1 -> 0.00 mm
- net SD3V3: track 37.8 -> 0.00 mm, vias 2 -> 0
- net D7: track 36.5 -> 0.00 mm
- net D8: track 33.9 -> 0.00 mm
- net D9: track 31.0 -> 0.00 mm
- net D10: track 28.2 -> 0.00 mm
- net GBUF: track 27.8 -> 0.00 mm, vias 2 -> 0
- net RAW: track 27.2 -> 0.00 mm, vias 1 -> 0
- net PWRBTN: track 26.6 -> 0.00 mm, vias 2 -> 0
- net SCK: track 26.1 -> 0.00 mm
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